File: pcb/power/power.kicad_pcb (KiCad board)
At the start: 2 copper layers, 114.3 x 74.9 mm, 27 parts, among them K1 CONN_3, P1 CONN_3X2, P2 CONN_4X2, T1 TRANSFORMER_F24-800-C2, U1 MC34063

Commit message: increased power CT capacitor size
It was determined that when the DC source
voltage is low (13.8 volts instead of 17 volts)
the MC34063 will regulate the output voltage
using a higher frequency.  And since a relatively
large inductor (L1, 220 uH) is being used this
can create a substantial voltage drop (1.5 V).

Z_L = 2*pi*f*L

To resolve this problem the timing capacitor (CT)
was doubled in size from 450 pF to 1000 pF.
Parts:
- C2: value 470 pF -> 1000 pF
Changed lines of the file:
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@@
       (effects (font (size 1.016 1.016) (thickness 0.2032)))
     )
-    (fp_text value "470 pF" (at 0 0) (layer F.SilkS) hide
+    (fp_text value "1000 pF" (at 0 0) (layer F.SilkS) hide
       (effects (font (size 1.016 1.016) (thickness 0.2032)))
     )
